File: CustomBoard.sch (KiCad schematic (older format))
At the start: 7 parts

Commit message: added deck expanders
Parts:
- removed U?: TPS731XX, symbol TPS731XX
- added C1: PowerC, symbol C_Small
- added J10: Sensor08, symbol Conn_01x05
- added J11: Sensor09, symbol Conn_01x05
- added J12: Sensor10, symbol Conn_01x05
- added J13: Sensor11, symbol Conn_01x05
- added J14: Sensor12, symbol Conn_01x05
- added J15: Sensor13, symbol Conn_01x05
- added J16: Sensor14, symbol Conn_01x05
- added J17: TEST_1P, symbol TEST_1P
- added J3: Sensor01, symbol Conn_01x05
- added J4: Sensor02, symbol Conn_01x05
- added J5: Sensor03, symbol Conn_01x05
- added J6: Sensor04, symbol Conn_01x05
- added J7: Sensor05, symbol Conn_01x05
- added J8: Sensor06, symbol Conn_01x05
- added J9: Sensor07, symbol Conn_01x05
- added R2, R3: 10k, symbol R
- R1: renamed from R?; value R -> 2k
- gave numbers to parts that had none: 5
Connections:
- net labels added: S01, S02, S03, S04, S05, S06, S07, S08, S09, S10, S11, S12, S13, S14, TEST
- net labels removed: CS0, CS1, CS2, CS3, MISO, MOSI, NRF1, NRF2, RX1, RX2, SCK, TX1, TX2, V2v8, VCOM, VUSB
- wire segments 14 -> 20
- no-connect marks 1 -> 17
Other:
- note added: "1-Wire Memory"
- note added: "ToF Expansion Slots"
- moved on the sheet: D1, R1, U1, U2

Commit message: pcb layout
Parts:
- C1: footprint (none) -> Capacitors_SMD:C_0603
- D1: footprint (none) -> LEDs:LED_0603
- J1, J2: footprint (none) -> Pin_Headers:Pin_Header_Straight_1x10_Pitch2.00mm
- J10, J11, J12, J13, J14, J15, J16, J3, J4, J5, J6, J7, J8, J9: footprint (none) -> Pin_Headers:Pin_Header_Straight_1x05_Pitch1.27mm
- J17: footprint (none) -> Measurement_Points:Measurement_Point_Round-SMD-Pad_Small
- R1, R2, R3: footprint (none) -> Resistors_SMD:R_0603
- U1: footprint (none) -> TO_SOT_Packages_SMD:SOT-23
- U2: footprint (none) -> Housings_DFN_QFN:QFN-24_4x4mm_Pitch0.5mm
Changed lines of the file:
@@
 F 0 "U2" H 5810 4230 60  0000 C CNN
 F 1 "PCA9555" H 5810 4460 60  0000 C CNN
-F 2 "" H 5810 4340 60  0001 C CNN
+F 2 "Housings_DFN_QFN:QFN-24_4x4mm_Pitch0.5mm" H 5810 4340 60  0001 C CNN
 F 3 "" H 5810 4340 60  0001 C CNN
 	1    5810 4340
@@
 F 0 "D1" H 4100 4065 50  0000 C CNN
 F 1 "POWER_LED" H 4100 3835 50  0000 C CNN
-F 2 "" H 4100 3965 50  0001 C CNN
+F 2 "LEDs:LED_0603" H 4100 3965 50  0001 C CNN
 F 3 "" H 4100 3965 50  0001 C CNN
 	1    4100 3965
@@
 F 0 "J1" H 910 7610 50  0000 C CNN
 F 1 "RIGHT" H 910 6510 50  0000 C CNN
-F 2 "" H 910 7110 50  0001 C CNN
+F 2 "Pin_Headers:Pin_Header_Straight_1x10_Pitch2.00mm" H 910 7110 50  0001 C CNN
 F 3 "" H 910 7110 50  0001 C CNN
 	1    910  7110
@@
 F 0 "J2" H 1730 7610 50  0000 C CNN
 F 1 "LEFT" H 1730 6510 50  0000 C CNN
-F 2 "" H 1730 7110 50  0001 C CNN
+F 2 "Pin_Headers:Pin_Header_Straight_1x10_Pitch2.00mm" H 1730 7110 50  0001 C CNN
 F 3 "" H 1730 7110 50  0001 C CNN
 	1    1730 7110
@@
 F 0 "U1" H 3770 7000 59  0000 C CNN
 F 1 "DS28E05" V 3615 7005 59  0000 C CNN
-F 2 "" H 3555 7150 79  0001 C CNN
+F 2 "TO_SOT_Packages_SMD:SOT-23" H 3555 7150 79  0001 C CNN
 F 3 "" H 3555 7150 79  0001 C CNN
 	1    3605 7000
@@
 F 0 "R1" V 3700 3965 50  0000 C CNN
 F 1 "2k" V 3615 3965 39  0000 C CNN
-F 2 "" V 3550 3965 50  0001 C CNN
+F 2 "Resistors_SMD:R_0603" V 3550 3965 50  0001 C CNN
 F 3 "" H 3620 3965 50  0001 C CNN
 	1    3620 3965
@@
 F 0 "R3" V 7075 3965 50  0000 C CNN
 F 1 "10k" V 6990 3965 39  0000 C CNN
-F 2 "" V 6925 3965 50  0001 C CNN
+F 2 "Resistors_SMD:R_0603" V 6925 3965 50  0001 C CNN
 F 3 "" H 6995 3965 50  0001 C CNN
 	1    6995 3965
@@
 F 0 "C1" V 950 815 50  0000 L CNN
 F 1 "PowerC" V 1085 650 50  0000 L CNN
-F 2 "" H 995 775 50  0001 C CNN
+F 2 "Capacitors_SMD:C_0603" H 995 775 50  0001 C CNN
 F 3 "" H 995 775 50  0001 C CNN
 	1    995  775
@@
 F 0 "R2" V 5815 2965 50  0000 C CNN
 F 1 "10k" V 5730 2965 39  0000 C CNN
-F 2 "" V 5665 2965 50  0001 C CNN
+F 2 "Resistors_SMD:R_0603" V 5665 2965 50  0001 C CNN
 F 3 "" H 5735 2965 50  0001 C CNN
 	1    5735 2965
@@
 F 0 "J9" H 8505 1400 50  0000 C CNN
 F 1 "Sensor07" H 8510 750 50  0000 C CNN
-F 2 "" H 8660 1080 50  0001 C CNN
+F 2 "Pin_Headers:Pin_Header_Straight_1x05_Pitch1.27mm" H 8660 1080 50  0001 C CNN
 F 3 "" H 8660 1080 50  0001 C CNN
 	1    8660 1080
@@
 F 0 "J10" H 8505 2230 50  0000 C CNN
 F 1 "Sensor08" H 8510 1580 50  0000 C CNN
-F 2 "" H 8660 1910 50  0001 C CNN
+F 2 "Pin_Headers:Pin_Header_Straight_1x05_Pitch1.27mm" H 8660 1910 50  0001 C CNN
 F 3 "" H 8660 1910 50  0001 C CNN
 	1    8660 1910
@@
 F 0 "J7" H 7840 1400 50  0000 C CNN
 F 1 "Sensor05" H 7845 750 50  0000 C CNN
-F 2 "" H 7995 1080 50  0001 C CNN
+F 2 "Pin_Headers:Pin_Header_Straight_1x05_Pitch1.27mm" H 7995 1080 50  0001 C CNN
 F 3 "" H 7995 1080 50  0001 C CNN
 	1    7995 1080
@@
 F 0 "J8" H 7840 2230 50  0000 C CNN
 F 1 "Sensor06" H 7845 1580 50  0000 C CNN
-F 2 "" H 7995 1910 50  0001 C CNN
+F 2 "Pin_Headers:Pin_Header_Straight_1x05_Pitch1.27mm" H 7995 1910 50  0001 C CNN
 F 3 "" H 7995 1910 50  0001 C CNN
 	1    7995 1910
@@
 F 0 "J5" H 7165 1400 50  0000 C CNN
 F 1 "Sensor03" H 7170 750 50  0000 C CNN
-F 2 "" H 7320 1080 50  0001 C CNN
+F 2 "Pin_Headers:Pin_Header_Straight_1x05_Pitch1.27mm" H 7320 1080 50  0001 C CNN
 F 3 "" H 7320 1080 50  0001 C CNN
 	1    7320 1080
@@
 F 0 "J6" H 7165 2230 50  0000 C CNN
 F 1 "Sensor04" H 7170 1580 50  0000 C CNN
-F 2 "" H 7320 1910 50  0001 C CNN
+F 2 "Pin_Headers:Pin_Header_Straight_1x05_Pitch1.27mm" H 7320 1910 50  0001 C CNN
 F 3 "" H 7320 1910 50  0001 C CNN
 	1    7320 1910
@@
 F 0 "J3" H 6500 1400 50  0000 C CNN
 F 1 "Sensor01" H 6505 750 50  0000 C CNN
-F 2 "" H 6655 1080 50  0001 C CNN
+F 2 "Pin_Headers:Pin_Header_Straight_1x05_Pitch1.27mm" H 6655 1080 50  0001 C CNN
 F 3 "" H 6655 1080 50  0001 C CNN
 	1    6655 1080
@@
 F 0 "J4" H 6500 2230 50  0000 C CNN
 F 1 "Sensor02" H 6505 1580 50  0000 C CNN
-F 2 "" H 6655 1910 50  0001 C CNN
+F 2 "Pin_Headers:Pin_Header_Straight_1x05_Pitch1.27mm" H 6655 1910 50  0001 C CNN
 F 3 "" H 6655 1910 50  0001 C CNN
 	1    6655 1910
@@
 F 0 "J11" H 9185 1400 50  0000 C CNN
 F 1 "Sensor09" H 9190 750 50  0000 C CNN
-F 2 "" H 9340 1080 50  0001 C CNN
+F 2 "Pin_Headers:Pin_Header_Straight_1x05_Pitch1.27mm" H 9340 1080 50  0001 C CNN
 F 3 "" H 9340 1080 50  0001 C CNN
 	1    9340 1080
@@
 F 0 "J12" H 9185 2230 50  0000 C CNN
 F 1 "Sensor10" H 9190 1580 50  0000 C CNN
-F 2 "" H 9340 1910 50  0001 C CNN
+F 2 "Pin_Headers:Pin_Header_Straight_1x05_Pitch1.27mm" H 9340 1910 50  0001 C CNN
 F 3 "" H 9340 1910 50  0001 C CNN
 	1    9340 1910
@@
 F 0 "J13" H 9845 1400 50  0000 C CNN
 F 1 "Sensor11" H 9850 750 50  0000 C CNN
-F 2 "" H 10000 1080 50  0001 C CNN
+F 2 "Pin_Headers:Pin_Header_Straight_1x05_Pitch1.27mm" H 10000 1080 50  0001 C CNN
 F 3 "" H 10000 1080 50  0001 C CNN
 	1    10000 1080
@@
 F 0 "J14" H 9845 2230 50  0000 C CNN
 F 1 "Sensor12" H 9850 1580 50  0000 C CNN
-F 2 "" H 10000 1910 50  0001 C CNN
+F 2 "Pin_Headers:Pin_Header_Straight_1x05_Pitch1.27mm" H 10000 1910 50  0001 C CNN
 F 3 "" H 10000 1910 50  0001 C CNN
 	1    10000 1910
@@
 F 0 "J15" H 10510 1400 50  0000 C CNN
 F 1 "Sensor13" H 10515 750 50  0000 C CNN
-F 2 "" H 10665 1080 50  0001 C CNN
+F 2 "Pin_Headers:Pin_Header_Straight_1x05_Pitch1.27mm" H 10665 1080 50  0001 C CNN
 F 3 "" H 10665 1080 50  0001 C CNN
 	1    10665 1080
@@
 F 0 "J16" H 10510 2230 50  0000 C CNN
 F 1 "Sensor14" H 10515 1580 50  0000 C CNN
-F 2 "" H 10665 1910 50  0001 C CNN
+F 2 "Pin_Headers:Pin_Header_Straight_1x05_Pitch1.27mm" H 10665 1910 50  0001 C CNN
 F 3 "" H 10665 1910 50  0001 C CNN
 	1    10665 1910
@@
 F 0 "J17" H 1770 835 50  0000 C CNN
 F 1 "TEST_1P" H 1705 965 50  0000 C CNN
-F 2 "" H 1905 765 50  0001 C CNN
+F 2 "Measurement_Points:Measurement_Point_Round-SMD-Pad_Small" H 1905 765 50  0001 C CNN
 F 3 "" H 1905 765 50  0001 C CNN
 	1    1705 765

Commit message: pcb layout update
Parts:
- J1: footprint Pin_Headers:Pin_Header_Straight_1x10_Pitch2.00mm -> Pin_Headers:Pin_Header_Straight_1x10_Pitch2.00mm_SMD_Pin1Right
- J10, J11, J12, J13, J14, J15, J16, J3, J4, J5, J6, J7, J8, J9: footprint Pin_Headers:Pin_Header_Straight_1x05_Pitch1.27mm -> footprint:SensorPads
- J2: footprint Pin_Headers:Pin_Header_Straight_1x10_Pitch2.00mm -> Pin_Headers:Pin_Header_Straight_1x10_Pitch2.00mm_SMD_Pin1Left
Changed lines of the file:
@@
 F 0 "J1" H 910 7610 50  0000 C CNN
 F 1 "RIGHT" H 910 6510 50  0000 C CNN
-F 2 "Pin_Headers:Pin_Header_Straight_1x10_Pitch2.00mm" H 910 7110 50  0001 C CNN
+F 2 "Pin_Headers:Pin_Header_Straight_1x10_Pitch2.00mm_SMD_Pin1Right" H 910 7110 50  0001 C CNN
 F 3 "" H 910 7110 50  0001 C CNN
 	1    910  7110
@@
 F 0 "J2" H 1730 7610 50  0000 C CNN
 F 1 "LEFT" H 1730 6510 50  0000 C CNN
-F 2 "Pin_Headers:Pin_Header_Straight_1x10_Pitch2.00mm" H 1730 7110 50  0001 C CNN
+F 2 "Pin_Headers:Pin_Header_Straight_1x10_Pitch2.00mm_SMD_Pin1Left" H 1730 7110 50  0001 C CNN
 F 3 "" H 1730 7110 50  0001 C CNN
 	1    1730 7110
@@
 F 0 "J9" H 8505 1400 50  0000 C CNN
 F 1 "Sensor07" H 8510 750 50  0000 C CNN
-F 2 "Pin_Headers:Pin_Header_Straight_1x05_Pitch1.27mm" H 8660 1080 50  0001 C CNN
+F 2 "footprint:SensorPads" H 8660 1080 50  0001 C CNN
 F 3 "" H 8660 1080 50  0001 C CNN
 	1    8660 1080
@@
 F 0 "J10" H 8505 2230 50  0000 C CNN
 F 1 "Sensor08" H 8510 1580 50  0000 C CNN
-F 2 "Pin_Headers:Pin_Header_Straight_1x05_Pitch1.27mm" H 8660 1910 50  0001 C CNN
+F 2 "footprint:SensorPads" H 8660 1910 50  0001 C CNN
 F 3 "" H 8660 1910 50  0001 C CNN
 	1    8660 1910
@@
 F 0 "J7" H 7840 1400 50  0000 C CNN
 F 1 "Sensor05" H 7845 750 50  0000 C CNN
-F 2 "Pin_Headers:Pin_Header_Straight_1x05_Pitch1.27mm" H 7995 1080 50  0001 C CNN
+F 2 "footprint:SensorPads" H 7995 1080 50  0001 C CNN
 F 3 "" H 7995 1080 50  0001 C CNN
 	1    7995 1080
@@
 F 0 "J8" H 7840 2230 50  0000 C CNN
 F 1 "Sensor06" H 7845 1580 50  0000 C CNN
-F 2 "Pin_Headers:Pin_Header_Straight_1x05_Pitch1.27mm" H 7995 1910 50  0001 C CNN
+F 2 "footprint:SensorPads" H 7995 1910 50  0001 C CNN
 F 3 "" H 7995 1910 50  0001 C CNN
 	1    7995 1910
@@
 F 0 "J5" H 7165 1400 50  0000 C CNN
 F 1 "Sensor03" H 7170 750 50  0000 C CNN
-F 2 "Pin_Headers:Pin_Header_Straight_1x05_Pitch1.27mm" H 7320 1080 50  0001 C CNN
+F 2 "footprint:SensorPads" H 7320 1080 50  0001 C CNN
 F 3 "" H 7320 1080 50  0001 C CNN
 	1    7320 1080
@@
 F 0 "J6" H 7165 2230 50  0000 C CNN
 F 1 "Sensor04" H 7170 1580 50  0000 C CNN
-F 2 "Pin_Headers:Pin_Header_Straight_1x05_Pitch1.27mm" H 7320 1910 50  0001 C CNN
+F 2 "footprint:SensorPads" H 7320 1910 50  0001 C CNN
 F 3 "" H 7320 1910 50  0001 C CNN
 	1    7320 1910
@@
 F 0 "J3" H 6500 1400 50  0000 C CNN
 F 1 "Sensor01" H 6505 750 50  0000 C CNN
-F 2 "Pin_Headers:Pin_Header_Straight_1x05_Pitch1.27mm" H 6655 1080 50  0001 C CNN
+F 2 "footprint:SensorPads" H 6655 1080 50  0001 C CNN
 F 3 "" H 6655 1080 50  0001 C CNN
 	1    6655 1080
@@
 F 0 "J4" H 6500 2230 50  0000 C CNN
 F 1 "Sensor02" H 6505 1580 50  0000 C CNN
-F 2 "Pin_Headers:Pin_Header_Straight_1x05_Pitch1.27mm" H 6655 1910 50  0001 C CNN
+F 2 "footprint:SensorPads" H 6655 1910 50  0001 C CNN
 F 3 "" H 6655 1910 50  0001 C CNN
 	1    6655 1910
@@
 F 0 "J11" H 9185 1400 50  0000 C CNN
 F 1 "Sensor09" H 9190 750 50  0000 C CNN
-F 2 "Pin_Headers:Pin_Header_Straight_1x05_Pitch1.27mm" H 9340 1080 50  0001 C CNN
+F 2 "footprint:SensorPads" H 9340 1080 50  0001 C CNN
 F 3 "" H 9340 1080 50  0001 C CNN
 	1    9340 1080
@@
 F 0 "J12" H 9185 2230 50  0000 C CNN
 F 1 "Sensor10" H 9190 1580 50  0000 C CNN
-F 2 "Pin_Headers:Pin_Header_Straight_1x05_Pitch1.27mm" H 9340 1910 50  0001 C CNN
+F 2 "footprint:SensorPads" H 9340 1910 50  0001 C CNN
 F 3 "" H 9340 1910 50  0001 C CNN
 	1    9340 1910
@@
 F 0 "J13" H 9845 1400 50  0000 C CNN
 F 1 "Sensor11" H 9850 750 50  0000 C CNN
-F 2 "Pin_Headers:Pin_Header_Straight_1x05_Pitch1.27mm" H 10000 1080 50  0001 C CNN
+F 2 "footprint:SensorPads" H 10000 1080 50  0001 C CNN
 F 3 "" H 10000 1080 50  0001 C CNN
 	1    10000 1080
@@
 F 0 "J14" H 9845 2230 50  0000 C CNN
 F 1 "Sensor12" H 9850 1580 50  0000 C CNN
-F 2 "Pin_Headers:Pin_Header_Straight_1x05_Pitch1.27mm" H 10000 1910 50  0001 C CNN
+F 2 "footprint:SensorPads" H 10000 1910 50  0001 C CNN
 F 3 "" H 10000 1910 50  0001 C CNN
 	1    10000 1910
@@
 F 0 "J15" H 10510 1400 50  0000 C CNN
 F 1 "Sensor13" H 10515 750 50  0000 C CNN
-F 2 "Pin_Headers:Pin_Header_Straight_1x05_Pitch1.27mm" H 10665 1080 50  0001 C CNN
+F 2 "footprint:SensorPads" H 10665 1080 50  0001 C CNN
 F 3 "" H 10665 1080 50  0001 C CNN
 	1    10665 1080
@@
 F 0 "J16" H 10510 2230 50  0000 C CNN
 F 1 "Sensor14" H 10515 1580 50  0000 C CNN
-F 2 "Pin_Headers:Pin_Header_Straight_1x05_Pitch1.27mm" H 10665 1910 50  0001 C CNN
+F 2 "footprint:SensorPads" H 10665 1910 50  0001 C CNN
 F 3 "" H 10665 1910 50  0001 C CNN
 	1    10665 1910

Commit message: 4m range ToF sensor parts
Parts:
- removed J17: TEST_1P, Measurement_Points:Measurement_Point_Round-SMD-Pad_Small, symbol TEST_1P
- removed R2, R3: 10k, Resistors_SMD:R_0603, symbol R
- added C2: 100n, symbol C_Small
- added C3: 4.7u, symbol C_Small
- added R4: 10k, symbol R
- added U3: VL53L1X, symbol VL53L1X
- C1: value PowerC -> 100n
Connections:
- net GND: now also U2.18 (A0), C2.2, C3.2, R4.2, U3.12 (GND4), U3.2 (AVSSS), U3.3 (GND1), U3.4 (GND2), U3.6 (GND3)
- net SCL: now also U3.10 (SCL)
- net SDA: now also U3.9 (SDA)
- net VCC: now also C2.1, C3.1, U3.1 (AVDDS), U3.11 (AVDD)
- net TEST renamed S15
- net S15: now also R4.1, U3.5 (XSHUT)
- net WKUP/OW renamed OW
- no-connect marks 17 -> 20
Other:
- note added: "Top ToF"
- moved on the sheet: U1
Changed lines of the file:
@@
 Title "CrazyFlie2.0"
 Date "2018-07-24"
-Rev ""
-Comp ""
+Rev "1.2"
+Comp "Group 14 FYP"
 Comment1 "Expansion Deck"
-Comment2 "VL53L0X Sensors"
-Comment3 ""
-Comment4 ""
+Comment2 "VL53L1X Sensors"
+Comment3 "15 Sensor SLAM"
+Comment4 "Obstacle Avoidance"
 $EndDescr
 $Comp
@@
 $EndComp
 Text GLabel 1110 6810 2    39   Input ~ 0
-WKUP/OW
+OW
 Text GLabel 1930 6610 2    39   Input ~ 0
 GND
@@
 	545  6215 545  7720
 Wire Notes Line
-	545  6215 4180 6215
+	545  6215 6700 6215
 Wire Notes Line
 	2420 6215 2420 7720
 Wire Notes Line
-	545  7720 4180 7720
+	545  7720 6700 7720
 Text Notes 575  6330 0    59   Italic 12
 IO EXPANDER
 $Comp
-L PWR_FLAG #FLG01
+L PWR_FLAG #FLG1
 U 1 1 5B5754C4
 P 725 720
-F 0 "#FLG01" H 725 795 50  0001 C CNN
+F 0 "#FLG1" H 725 795 50  0001 C CNN
 F 1 "PWR_FLAG" H 725 870 50  0000 C CNN
 F 2 "" H 725 720 50  0001 C CNN
@@
 $EndComp
 $Comp
-L PWR_FLAG #FLG02
+L PWR_FLAG #FLG2
 U 1 1 5B575536
 P 1245 720
-F 0 "#FLG02" H 1245 795 50  0001 C CNN
+F 0 "#FLG2" H 1245 795 50  0001 C CNN
 F 1 "PWR_FLAG" H 1245 870 50  0000 C CNN
 F 2 "" H 1245 720 50  0001 C CNN
@@
 VCC
 Wire Wire Line
-	1245 810  1245 720
+	1245 720  1245 810
 Wire Wire Line
 	725  720  725  805
@@
 Wire Wire Line
 	5585 3550 5585 3430
-Wire Wire Line
-	5585 3430 5435 3430
-Connection ~ 5435 3430
 $Comp
 L DS28E05 U1
 U 1 1 5B575B36
-P 3605 7000
-F 0 "U1" H 3770 7000 59  0000 C CNN
-F 1 "DS28E05" V 3615 7005 59  0000 C CNN
-F 2 "TO_SOT_Packages_SMD:SOT-23" H 3555 7150 79  0001 C CNN
-F 3 "" H 3555 7150 79  0001 C CNN
-	1    3605 7000
-	1    0    0    -1
-$EndComp
-NoConn ~ 3140 7000
-Text GLabel 3005 7140 0    39   Input ~ 0
-GND
-Text GLabel 3005 6850 0    39   Input ~ 0
-WKUP/OW
-Wire Wire Line
-	3005 6850 3140 6850
-Wire Wire Line
-	3140 7140 3005 7140
+P 3525 7005
+F 0 "U1" H 3690 7005 59  0000 C CNN
+F 1 "DS28E05" V 3535 7010 59  0000 C CNN
+F 2 "TO_SOT_Packages_SMD:SOT-23" H 3475 7155 79  0001 C CNN
+F 3 "" H 3475 7155 79  0001 C CNN
+	1    3525 7005
+	1    0    0    -1
+$EndComp
+NoConn ~ 3060 7005
+Text GLabel 2925 7145 0    39   Input ~ 0
+GND
+Text GLabel 2925 6855 0    39   Input ~ 0
+OW
+Wire Wire Line
+	2925 6855 3060 6855
+Wire Wire Line
+	3060 7145 2925 7145
 Text GLabel 6185 3310 1    39   Input ~ 0
 SCL
@@
 Wire Wire Line
 	5885 3310 5885 3550
-Text GLabel 7340 3965 2    39   Input ~ 0
-VCC
-$Comp
-L R R3
-U 1 1 5B573F58
-P 6995 3965
-F 0 "R3" V 7075 3965 50  0000 C CNN
-F 1 "10k" V 6990 3965 39  0000 C CNN
-F 2 "Resistors_SMD:R_0603" V 6925 3965 50  0001 C CNN
-F 3 "" H 6995 3965 50  0001 C CNN
-	1    6995 3965
-	0    -1   -1   0
-$EndComp
-Wire Wire Line
-	6845 3965 6600 3965
-Wire Wire Line
-	7145 3965 7340 3965
 $Comp
 L C_Small C1
 U 1 1 5B574396
 P 995 775
-F 0 "C1" V 950 815 50  0000 L CNN
-F 1 "PowerC" V 1085 650 50  0000 L CNN
+F 0 "C1" V 950 815 39  0000 L CNN
+F 1 "100n" V 1100 705 39  0000 L CNN
 F 2 "Capacitors_SMD:C_0603" H 995 775 50  0001 C CNN
 F 3 "" H 995 775 50  0001 C CNN
@@
 	1095 775  1245 775
 Connection ~ 1245 775
-$Comp
-L R R2
-U 1 1 5B57494F
-P 5735 2965
-F 0 "R2" V 5815 2965 50  0000 C CNN
-F 1 "10k" V 5730 2965 39  0000 C CNN
-F 2 "Resistors_SMD:R_0603" V 5665 2965 50  0001 C CNN
-F 3 "" H 5735 2965 50  0001 C CNN
-	1    5735 2965
-	-1   0    0    1
-$EndComp
-Wire Wire Line
-	5735 3115 5735 3550
-Text GLabel 5735 2680 1    39   Input ~ 0
-VCC
-Wire Wire Line
-	5735 2680 5735 2815
 NoConn ~ 11060 4010
 $Comp
@@
 S14
 Text GLabel 6600 4115 2    39   Input ~ 0
-TEST
+S15
 Wire Notes Line
 	4180 7720 4180 6215
@@
 NoConn ~ 1110 7210
 NoConn ~ 1110 7110
-Text GLabel 1705 810  3    39   Input ~ 0
-TEST
-$Comp
-L TEST_1P J17
-U 1 1 5B57BB06
-P 1705 765
-F 0 "J17" H 1770 835 50  0000 C CNN
-F 1 "TEST_1P" H 1705 965 50  0000 C CNN
-F 2 "Measurement_Points:Measurement_Point_Round-SMD-Pad_Small" H 1905 765 50  0001 C CNN
-F 3 "" H 1905 765 50  0001 C CNN
-	1    1705 765
-	1    0    0    -1
-$EndComp
-Wire Wire Line
-	1705 810  1705 765
+$Comp
+L VL53L1X U3
+U 1 1 5B58A20A
+P 5745 6965
+F 0 "U3" H 5745 6555 60  0000 C CNN
+F 1 "VL53L1X" H 5745 7395 60  0000 C CNN
+F 2 "" H 5745 6965 60  0001 C CNN
+F 3 "" H 5745 6965 60  0001 C CNN
+	1    5745 6965
+	1    0    0    -1
+$EndComp
+Text GLabel 4755 7125 0    39   Input ~ 0
+S15
+$Comp
+L R R4
+U 1 1 5B58A900
+P 4875 7425
+F 0 "R4" V 4955 7425 50  0000 C CNN
+F 1 "10k" V 4875 7425 39  0000 C CNN
+F 2 "" V 4805 7425 50  0001 C CNN
+F 3 "" H 4875 7425 50  0001 C CNN
+	1    4875 7425
+	1    0    0    -1
+$EndComp
+Wire Wire Line
+	4755 7125 5225 7125
+NoConn ~ 6265 7225
+Wire Wire Line
+	4755 6420 6490 6420
+Wire Wire Line
+	6490 6420 6490 6915
+Wire Wire Line
+	6490 6915 6265 6915
+$Comp
+L C_Small C2
+U 1 1 5B58B483
+P 4830 6610
+F 0 "C2" H 4735 6680 39  0000 L CNN
+F 1 "100n" H 4665 6550 39  0000 L CNN
+F 2 "" H 4830 6610 50  0001 C CNN
+F 3 "" H 4830 6610 50  0001 C CNN
+	1    4830 6610
+	1    0    0    -1
+$EndComp
+Wire Wire Line
+	4830 6915 5225 6915
+Wire Wire Line
+	4525 7020 5225 7020
+Wire Wire Line
+	5225 7225 5100 7225
+Wire Wire Line
+	5100 7225 5100 7655
+Wire Wire Line
+	4525 7655 6570 7655
+Wire Wire Line
+	4875 7275 4875 7125
+Connection ~ 4875 7125
+Wire Wire Line
+	4875 7655 4875 7575
+Wire Wire Line
+	4525 7655 4525 7020
+Connection ~ 4875 7655
+Text GLabel 6265 6810 2    39   Input ~ 0
+SCL
+Text GLabel 6265 7020 2    39   Input ~ 0
+SDA
+NoConn ~ 6265 7120
+Wire Wire Line
+	6265 6700 6570 6700
+Wire Wire Line
+	6570 6700 6570 7655
+Connection ~ 5100 7655
+Text GLabel 4755 6420 0    39   Input ~ 0
+VCC
+Text GLabel 4760 6810 0    39   Input ~ 0
+GND
+Wire Wire Line
+	5225 6700 5190 6700
+Wire Wire Line
+	5190 6700 5190 6420
+Connection ~ 5190 6420
+$Comp
+L C_Small C3
+U 1 1 5B58DF49
+P 5050 6610
+F 0 "C3" H 4960 6680 39  0000 L CNN
+F 1 "4.7u" H 4915 6550 39  0000 L CNN
+F 2 "" H 5050 6610 50  0001 C CNN
+F 3 "" H 5050 6610 50  0001 C CNN
+	1    5050 6610
+	1    0    0    -1
+$EndComp
+Wire Wire Line
+	4830 6510 4830 6420
+Connection ~ 4830 6420
+Wire Wire Line
+	5050 6420 5050 6510
+Connection ~ 5050 6420
+Wire Wire Line
+	4830 6710 4830 7020
+Connection ~ 4830 7020
+Connection ~ 4830 6915
+Wire Wire Line
+	5050 6710 5050 6915
+Connection ~ 5050 6915
+Wire Wire Line
+	4760 6810 5225 6810
+Connection ~ 4830 6810
+Connection ~ 5050 6810
+Wire Notes Line
+	6700 7720 6700 6215
+Text Notes 4240 6335 0    59   Italic 12
+Top ToF
+NoConn ~ 5735 3550
+Text GLabel 6600 3965 2    39   Input ~ 0
+GND
+Wire Wire Line
+	5585 3430 5435 3430
+Connection ~ 5435 3430
 $EndSCHEMATC

Commit message: new footprints
Parts:
- C1: footprint Capacitors_SMD:C_0603 -> Capacitors_SMD:C_0402
- C2, C3: footprint (none) -> Capacitors_SMD:C_0402
- D1: footprint LEDs:LED_0603 -> LEDs:LED_0402
- R1: footprint Resistors_SMD:R_0603 -> Resistors_SMD:R_0402
- R4: footprint (none) -> Resistors_SMD:R_0402
- U3: footprint (none) -> footprint:VL53L1X
Changed lines of the file:
@@
 F 0 "D1" H 4100 4065 50  0000 C CNN
 F 1 "POWER_LED" H 4100 3835 50  0000 C CNN
-F 2 "LEDs:LED_0603" H 4100 3965 50  0001 C CNN
+F 2 "LEDs:LED_0402" H 4100 3965 50  0001 C CNN
 F 3 "" H 4100 3965 50  0001 C CNN
 	1    4100 3965
@@
 IO EXPANDER
 $Comp
-L PWR_FLAG #FLG1
+L PWR_FLAG #FLG01
 U 1 1 5B5754C4
 P 725 720
-F 0 "#FLG1" H 725 795 50  0001 C CNN
+F 0 "#FLG01" H 725 795 50  0001 C CNN
 F 1 "PWR_FLAG" H 725 870 50  0000 C CNN
 F 2 "" H 725 720 50  0001 C CNN
@@
 $EndComp
 $Comp
-L PWR_FLAG #FLG2
+L PWR_FLAG #FLG02
 U 1 1 5B575536
 P 1245 720
-F 0 "#FLG2" H 1245 795 50  0001 C CNN
+F 0 "#FLG02" H 1245 795 50  0001 C CNN
 F 1 "PWR_FLAG" H 1245 870 50  0000 C CNN
 F 2 "" H 1245 720 50  0001 C CNN
@@
 F 0 "R1" V 3700 3965 50  0000 C CNN
 F 1 "2k" V 3615 3965 39  0000 C CNN
-F 2 "Resistors_SMD:R_0603" V 3550 3965 50  0001 C CNN
+F 2 "Resistors_SMD:R_0402" V 3550 3965 50  0001 C CNN
 F 3 "" H 3620 3965 50  0001 C CNN
 	1    3620 3965
@@
 F 0 "C1" V 950 815 39  0000 L CNN
 F 1 "100n" V 1100 705 39  0000 L CNN
-F 2 "Capacitors_SMD:C_0603" H 995 775 50  0001 C CNN
+F 2 "Capacitors_SMD:C_0402" H 995 775 50  0001 C CNN
 F 3 "" H 995 775 50  0001 C CNN
 	1    995  775
@@
 F 0 "U3" H 5745 6555 60  0000 C CNN
 F 1 "VL53L1X" H 5745 7395 60  0000 C CNN
-F 2 "" H 5745 6965 60  0001 C CNN
+F 2 "footprint:VL53L1X" H 5745 6965 60  0001 C CNN
 F 3 "" H 5745 6965 60  0001 C CNN
 	1    5745 6965
@@
 F 0 "R4" V 4955 7425 50  0000 C CNN
 F 1 "10k" V 4875 7425 39  0000 C CNN
-F 2 "" V 4805 7425 50  0001 C CNN
+F 2 "Resistors_SMD:R_0402" V 4805 7425 50  0001 C CNN
 F 3 "" H 4875 7425 50  0001 C CNN
 	1    4875 7425
@@
 F 0 "C2" H 4735 6680 39  0000 L CNN
 F 1 "100n" H 4665 6550 39  0000 L CNN
-F 2 "" H 4830 6610 50  0001 C CNN
+F 2 "Capacitors_SMD:C_0402" H 4830 6610 50  0001 C CNN
 F 3 "" H 4830 6610 50  0001 C CNN
 	1    4830 6610
@@
 F 0 "C3" H 4960 6680 39  0000 L CNN
 F 1 "4.7u" H 4915 6550 39  0000 L CNN
-F 2 "" H 5050 6610 50  0001 C CNN
+F 2 "Capacitors_SMD:C_0402" H 5050 6610 50  0001 C CNN
 F 3 "" H 5050 6610 50  0001 C CNN
 	1    5050 6610
