File: OneToF.sch (KiCad schematic (older format))
At the start: 5 parts, among them J19 Top, J20 Bot, U5 VL53L1X

Commit message: update
Changed lines of the file:
@@
 AR Path="/5B640D2F/5B646238/5B642FEB" Ref="U18"  Part="1"
 AR Path="/5B640D2F/5B64623D/5B642FEB" Ref="U19"  Part="1"
-F 0 "U16" H 5465 3645 60  0000 C CNN
+F 0 "U19" H 5465 3645 60  0000 C CNN
 F 1 "VL53L1X" H 5465 4485 60  0000 C CNN
 F 2 "footprint:VL53L1X" H 5465 4055 60  0001 C CNN
@@
 AR Path="/5B640D2F/5B646238/5B642FEC" Ref="C34"  Part="1"
 AR Path="/5B640D2F/5B64623D/5B642FEC" Ref="C36"  Part="1"
-F 0 "C30" H 4580 3715 39  0000 L CNN
+F 0 "C36" H 4580 3715 39  0000 L CNN
 F 1 "4.7u" H 4580 3565 39  0000 L CNN
 F 2 "Capacitors_SMD:C_0402" H 4570 3645 50  0001 C CNN
@@
 AR Path="/5B640D2F/5B646238/5B642FED" Ref="C33"  Part="1"
 AR Path="/5B640D2F/5B64623D/5B642FED" Ref="C35"  Part="1"
-F 0 "C29" H 4360 3710 39  0000 L CNN
+F 0 "C35" H 4360 3710 39  0000 L CNN
 F 1 "100n" H 4360 3560 39  0000 L CNN
 F 2 "Capacitors_SMD:C_0402" H 4350 3640 50  0001 C CNN
@@
 AR Path="/5B640D2F/5B646238/5B642FEE" Ref="J45"  Part="1"
 AR Path="/5B640D2F/5B64623D/5B642FEE" Ref="J47"  Part="1"
-F 0 "J41" H 6935 3825 50  0000 C CNN
+F 0 "J47" H 6935 3825 50  0000 C CNN
 F 1 "Top" H 6935 3525 50  0000 C CNN
 F 2 "footprint:ToFTop" H 6935 3725 50  0001 C CNN
@@
 AR Path="/5B640D2F/5B646238/5B642FEF" Ref="J46"  Part="1"
 AR Path="/5B640D2F/5B64623D/5B642FEF" Ref="J48"  Part="1"
-F 0 "J42" H 6935 4515 50  0000 C CNN
+F 0 "J48" H 6935 4515 50  0000 C CNN
 F 1 "Bot" H 6935 4115 50  0000 C CNN
 F 2 "footprint:ToFBottom" H 6935 4315 50  0001 C CNN
