File: Camera/Camera.kicad_pcb (KiCad board)
At the start: 2 copper layers, 15.6 x 13.8 mm, 11 parts, among them J1 PulCon, J2 IntCon, J3 Camera, U1 AMG8833

Commit message: reformatting
Parts:
- moved J2 1.88 mm to (158.4, 101.6)
- moved J1 1.23 mm to (158.4, 94.8)
- moved R3 1.19 mm to (154.4, 95.0)
- moved R1 1.08 mm to (154.4, 100.4)
- moved R2 1.05 mm to (154.4, 97.7)
- moved J3 0.85 mm to (154.0, 98.2)
- moved R4 0.68 mm to (164.9, 99.0), turned to 90 degrees
- moved C2 0.12 mm to (164.2, 102.8)
Routing:
- net SDA: track 7.69 -> 5.96 mm
- net Net-(J1-Pad2): track 11.1 -> 9.89 mm
- net Net-(C2-Pad2): track 4.43 -> 3.38 mm
- net Net-(C2-Pad1): track 6.39 -> 5.46 mm
- net GND: track 24.2 -> 24.7 mm
Other:
- board size 15.6 x 13.8 mm -> 14.8 x 13.9 mm
- board text added: "AMG8833 Thermal Camera"
- board text added: "INT Enable"
- board text added: "PULL Enable"
